File: Net4CPC.sch (EAGLE design)
At the start: 22 parts, among them CON1 CPCBUS, IC1 74LS30N, IC2 74LS32N, IC3 74LS32N, IC4 AMS1117-3.3

Commit message: Add files via upload
Electrolytic capacitors value change
Parts:
- C4, C5: value 1uF/16V -> 10uF/16V
Changed lines of the file:
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@@
 <part name="P+4" library="supply1" library_urn="urn:adsk.eagle:library:371" deviceset="+5V" device=""/>
 <part name="IC4" library="SparkFun" deviceset="V_REG_LM1117" device="SOT223" value="AMS1117-3.3"/>
-<part name="C4" library="rcl" library_urn="urn:adsk.eagle:library:334" deviceset="CPOL-EU" device="E5-6" package3d_urn="urn:adsk.eagle:package:23368/1" value="1uF/16V"/>
-<part name="C5" library="rcl" library_urn="urn:adsk.eagle:library:334" deviceset="CPOL-EU" device="E5-6" package3d_urn="urn:adsk.eagle:package:23368/1" value="1uF/16V"/>
+<part name="C4" library="rcl" library_urn="urn:adsk.eagle:library:334" deviceset="CPOL-EU" device="E5-6" package3d_urn="urn:adsk.eagle:package:23368/1" value="10uF/16V"/>
+<part name="C5" library="rcl" library_urn="urn:adsk.eagle:library:334" deviceset="CPOL-EU" device="E5-6" package3d_urn="urn:adsk.eagle:package:23368/1" value="10uF/16V"/>
 </parts>
 <sheets>
